Commit message: adding to urdf

File: src/bevbot_arduino/description/urdf/bevbot_core.xacro (robot description, xacro)
@@ -19,9 +19,17 @@
   <link name="${prefix}base_link">
   </link>
+ <!-- Base footprint Link =============================================================================================-->
+  <joint name="base_footprint_joint" type="fixed">
+    <parent link="${prefix}base_link"/>
+    <child link="${prefix}base_footprint"/>
+    <origin xyz="0 0 0"/>
+  </joint>
+  <link name="${prefix}base_footprint">
+  </link>
   <!-- Chassis link ====================================================================================-->
   <joint name="${prefix}chassis_joint" type="fixed">
     <parent link="${prefix}base_link"/>
     <child link="${prefix}chassis"/>
-    <origin xyz="-.0623 0 0"/>
+    <origin xyz="0 0 0"/>
   </joint>
   <link name="${prefix}chassis">

Commit message: testing at my house

File: src/bevbot_arduino/description/urdf/bevbot_core.xacro (robot description, xacro)
@@ -19,5 +19,5 @@
   <xacro:property name="wheel_len" value="0.0127" />
   <xacro:property name="wheel_space" value="0.0127" />
-  <xacro:property name="wheel_radius" value="0.04445" />
+  <xacro:property name="wheel_radius" value="0.0460375" />
   <xacro:property name="caster_wheel_mass" value="0.1" /> <!-- arbitrary value for caster wheel mass -->
   <xacro:property name="caster_wheel_radius" value="0.0508" />

Commit message: navigation using nav2 stack works and is tested

File: src/bevbot_arduino/description/urdf/bevbot_core.xacro (robot description, xacro)
@@ -19,5 +19,5 @@
   <xacro:property name="wheel_len" value="0.0127" />
   <xacro:property name="wheel_space" value="0.0127" />
-  <xacro:property name="wheel_radius" value="0.0460375" />
+  <xacro:property name="wheel_radius" value="0.0460375"  />   <!---"0.0460375"  old value-->
   <xacro:property name="caster_wheel_mass" value="0.1" /> <!-- arbitrary value for caster wheel mass -->
   <xacro:property name="caster_wheel_radius" value="0.0508" />
